File: _autosave-matrixboardproto1.kicad_sch (KiCad schematic)
At the start: 12 parts, among them Q1 BC107, SW1 SW_Push

Commit message: Add files via upload
Parts:
- removed D1: LED, symbol Device:LED
- removed SW1: SW_Push, symbol Switch:SW_Push
- added D2: LED, symbol Device:LED
- added J1: Barrel_Jack, symbol Connector:Barrel_Jack
- added Waveshare Matrix1: Waveshare Matrix, Waveshare Matrix, symbol Matrix_Board_Lib:Waveshare_LED_Matrix
Connections:
- net +12V: now also D2.2 (A), J1.1
- net +5V: now also A1.5V1 (5V), A1.5V3 (5V), R2.2, U Ultrasonic1. (Vcc), Waveshare Matrix1. (R2); no longer A1.VIN
- net GND: now also J1.2, Waveshare Matrix1. (R2)
- net at A1.A1: no longer U Ultrasonic1. (Vcc)
- new net: A1.VIN, D2.1 (K), U 12v-5v Regulator1. (Out-)
- now unconnected: A1.A2, R1.2
