File: matrixboardproto1.kicad_pcb (KiCad board)
At the start: 2 copper layers, 122.5 x 60 mm, 25 parts, among them J1 Waveshare_Input_Conn, J2 Ultrasonic_Conn, J3 PJ-102AH, J4 LED_Switch_Conn, J5 Debug_Conn, J6 Button_Conn, J7 Button_Conn, J9 WAVESHARE_PWR, Q1 2N2222

Commit message: Add files via upload
Parts:
- moved J1 19.6 mm to (202.5, 73.5), turned to 180 degrees
- moved LS1 0.50 mm to (233.0, 86.5)
- turned R1 to 180 degrees
- turned R3 to 0 degrees
- turned R5 to -90 degrees
- turned R6 to -90 degrees
Connections:
- A** pad 5V1: (no net) -> +5V
- A** pad 5V2: (no net) -> +5V
- A** pad 5V3: (no net) -> +5V
- A** pad 5V4: (no net) -> +5V
- A** pad A0: (no net) -> /A
- A** pad A1: (no net) -> /B
- A** pad A2: (no net) -> /C
- A** pad A3: (no net) -> /D
- A** pad A4: (no net) -> /E
- A** pad D1: (no net) -> /Speaker_PWM
- A** pad D10: (no net) -> /LAT
- A** pad D11: (no net) -> /CLK
- A** pad D2: (no net) -> Net-(D3-A)
- A** pad D24: (no net) -> /R1
- A** pad D25: (no net) -> /G1
- A** pad D26: (no net) -> /B1
- A** pad D27: (no net) -> /R2
- A** pad D28: (no net) -> /G2
- A** pad D29: (no net) -> /B2
- A** pad D3: (no net) -> Net-(D2-A)
- A** pad D4: (no net) -> Net-(D1-A)
- A** pad D9: (no net) -> /OE
- A** pad GND2: (no net) -> GND
- A** pad GND3: (no net) -> GND
- A** pad GND5: (no net) -> GND
- A** pad GND6: (no net) -> GND
- A** pad VIN: (no net) -> /12V_SWITCH
- J9 pad 1: +5V -> +5V_Matrix
- J9 pad 2: +5V -> +5V_Matrix
Routing:
- net GND: track 0.00 -> 325.8 mm, vias 0 -> 2
- net +5V_Matrix: track 0.00 -> 179.0 mm
- net /12V_SWITCH: track 0.00 -> 167.4 mm
- net +5V: track 0.00 -> 102.6 mm, vias 0 -> 2
- net /OE: track 0.00 -> 77.2 mm
- net /CLK: track 0.00 -> 72.7 mm
- net /LAT: track 0.00 -> 72.5 mm
- net /A: track 0.00 -> 56.8 mm
- net /B: track 0.00 -> 56.5 mm
- net /E: track 0.00 -> 55.7 mm
- net /C: track 0.00 -> 50.1 mm
- net /D: track 0.00 -> 49.2 mm
- net /Speaker_PWM: track 0.00 -> 37.4 mm, vias 0 -> 2
- net Net-(LS1-Pin_1): track 0.00 -> 34.7 mm
- net +12V: track 0.00 -> 31.6 mm
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