File: matrixboardproto1.kicad_sch (KiCad schematic)
At the start: 11 parts, among them Q1 BC107, SW1 SW_Push

Commit message: Add files via upload
Parts:
- removed SW1: SW_Push, symbol Switch:SW_Push
- added A1: Arduino_Mega2560_R3_Shield, PCM_arduino-library:Arduino_Mega2560_R3_Shield, symbol arduino-library:Arduino_Mega2560_R3_Shield
- added D2: LED, symbol Device:LED
- renumbered D1 to Waveshare
Connections:
- net +12V: now also D2.2 (A)
- net GND: now also A1.GND1 (GND)
- net at R1.2: now also R2.2
- new net: D2.1 (K), U 12v-5v Regulator1. (Out-)
- new net +5V: U 12v-5v Regulator1. (Out-), Waveshare.2 (A)
Other:
- moved on the sheet: C1, C2, LS1, Q1, R1, R2, R3, U Ultrasonic1, Waveshare

Commit message: Add files via upload
Parts:
- removed Waveshare: LED, symbol Device:LED
- added J1: Barrel_Jack, symbol Connector:Barrel_Jack
- added Waveshare Matrix1: Waveshare Matrix, Waveshare Matrix, symbol Matrix_Board_Lib:Waveshare_LED_Matrix
Connections:
- net GND is gone; now on net +5V: A1.GND1 (GND), C1.1, LS1.2, Q1.1 (E), U 12v-5v Regulator1. (Out-), U Ultrasonic1. (Vcc)
- net +12V: now also J1.1
- net +5V: now also A1.5V1 (5V), A1.5V3 (5V), R2.2, J1.2, Waveshare Matrix1. (R2)
- net at D2.1 (K), U 12v-5v Regulator1. (Out-): now also A1.VIN
- net at R1.2: now also A1.D31; no longer R2.2
- net at A1.A0: now also Waveshare Matrix1. (R2)
- net at A1.A1: now also Waveshare Matrix1. (R2)
- net at A1.A2: now also Waveshare Matrix1. (R2)
- net at A1.A3: now also Waveshare Matrix1. (R2)
- net at A1.A4: now also Waveshare Matrix1. (R2)
- net at A1.D10: now also Waveshare Matrix1. (R2)
- net at A1.D11: now also Waveshare Matrix1. (R2)
- net at A1.D24: now also Waveshare Matrix1. (R2)
- net at A1.D25: now also Waveshare Matrix1. (R2)
- net at A1.D26: now also Waveshare Matrix1. (R2)
- net at A1.D27: now also Waveshare Matrix1. (R2)
- net at A1.D28: now also Waveshare Matrix1. (R2)
- net at A1.D29: now also Waveshare Matrix1. (R2)
- net at A1.D34: now also U Ultrasonic1. (Vcc)
- net at A1.D35: now also U Ultrasonic1. (Vcc)
- net at A1.D9: now also Waveshare Matrix1. (R2)
Other:
- moved on the sheet: C1, C2, LS1, Q1, R1, R2, R3, U Ultrasonic1

Commit message: Add files via upload
Parts:
- removed J1: Barrel_Jack, symbol Connector:Barrel_Jack
- removed U 12v-5v Regulator1: ~, symbol Matrix_Board_Lib:DFR0831
- removed U Ultrasonic1: ~, symbol Matrix_Board_Lib:HCSR04_
- removed Waveshare Matrix1: Waveshare Matrix, Waveshare Matrix, symbol Matrix_Board_Lib:Waveshare_LED_Matrix
- added D1, D3: LED, LED_THT:LED_D5.0mm_Horizontal_O6.35mm_Z15.0mm, symbol Device:LED
- added J1: Waveshare_Input_Conn, Connector_IDC:IDC-Header_2x08_P2.54mm_Vertical, symbol Connector_Generic:Conn_02x08_Odd_Even
- added J2: Ultrasonic_Conn, Connector_PinHeader_1.00mm:PinHeader_1x04_P1.00mm_Vertical, symbol Connector_Generic:Conn_01x04
- added J3: Barrel_Jack_Switch_Pin3Ring, Connector_BarrelJack:BarrelJack_GCT_DCJ200-10-A_Horizontal, symbol Connector:Barrel_Jack_Switch_Pin3Ring
- added J4: LED_Switch_Conn, Connector:FanPinHeader_1x03_P2.54mm_Vertical, symbol Connector_Generic:Conn_01x03
- added J5: Debug_Conn, symbol Connector_Generic:Conn_01x06
- added J6: Button0, Connector_PinHeader_1.00mm:PinHeader_1x02_P1.00mm_Vertical, symbol Connector_Generic:Conn_01x02
- added J7: Button1, Connector_PinHeader_1.00mm:PinHeader_1x02_P1.00mm_Vertical, symbol Connector_Generic:Conn_01x02
- added J8: Waveshare_PWR, Connector_PinHeader_1.00mm:PinHeader_1x02_P1.00mm_Vertical, symbol Connector_Generic:Conn_01x02
- added R4, R5, R6: R600, Resistor_SMD:R_0805_2012Metric_Pad1.20x1.40mm_HandSolder, symbol Device:R
- added R7, R8: R10k, Resistor_SMD:R_0805_2012Metric_Pad1.20x1.40mm_HandSolder, symbol Device:R
- added U1: ~, matrixboard:DFR_Regulator, symbol Matrix_Board_Lib:DFR0831
- C1: value C -> 1nF; footprint (none) -> Capacitor_SMD:C_0805_2012Metric_Pad1.18x1.45mm_HandSolder
- C2: value C -> 10nF; footprint (none) -> Capacitor_SMD:C_0805_2012Metric_Pad1.18x1.45mm_HandSolder
- D2: footprint (none) -> LED_THT:LED_D5.0mm_Horizontal_O6.35mm_Z15.0mm
- LS1: footprint (none) -> Buzzer_Beeper:Speaker_CUI_CMR-1206S-67
- Q1: value BC107 -> 2N2222
- R1: value R -> R220; footprint (none) -> Resistor_SMD:R_0805_2012Metric_Pad1.20x1.40mm_HandSolder
- R2: value R -> R20; footprint (none) -> Resistor_SMD:R_0805_2012Metric_Pad1.20x1.40mm_HandSolder
- R3: value R -> R100; footprint (none) -> Resistor_SMD:R_0805_2012Metric_Pad1.20x1.40mm_HandSolder
Connections:
- net +12V: now also J3.1, J4.1 (Pin_1), J4.2 (Pin_2), U1.1 (IN-); no longer D2.2 (A)
- net at D2.1 (K): now also R5.1; no longer A1.VIN
- net A: now reaches A1.A0
- net A: now also J1.8 (Pin_8)
- net B: now reaches A1.A1
- net B: now also J1.7 (Pin_7)
- net C: now reaches A1.A2
- net C: now also J1.6 (Pin_6)
- net D: now reaches A1.A3
- net D: now also J1.5 (Pin_5)
- net E: now reaches A1.A4
- net E: now also J1.9 (Pin_9)
- net LAT: now reaches A1.D10
- net LAT: now also J1.3 (Pin_3)
- net CLK: now reaches A1.D11
- net CLK: now also J1.4 (Pin_4)
- net R1: now reaches A1.D24
- net R1: now also A1.D27, J1.16 (Pin_16)
- net G1: now reaches A1.D25
- net G1: now also J1.15 (Pin_15)
- net B1: now reaches A1.D26
- net B1: now also J1.14 (Pin_14)
- net G2: now reaches A1.D28
- net G2: now also J1.11 (Pin_11)
- net B2: now reaches A1.D29
- net B2: now also J1.10 (Pin_10)
- net OE: now reaches A1.D9
- net OE: now also J1.2 (Pin_2)
- net at A1.D31: no longer R1.2
- net Button0: now reaches A1.D13
- net Button0: now also J6.1 (Pin_1)
- net Button1: now reaches A1.D22
- net Button1: now also J7.1 (Pin_1)
- net Trig: now reaches A1.D32
- net Trig: now also J2.2 (Pin_2)
- net Echo: now reaches A1.D33
- net Echo: now also J2.3 (Pin_3)
- net at A1.D36: now also J5.1 (Pin_1)
- net at A1.D37: now also J5.2 (Pin_2)
- net at A1.D38: now also J5.3 (Pin_3)
- net at A1.D39: now also J5.4 (Pin_4)
- net at A1.D40: now also J5.5 (Pin_5)
- net Speaker_PWM: now reaches A1.D44
- net Speaker_PWM: now also R1.2
- net at A1.D47: now also D1.2 (A)
- net at A1.D48: now also D2.2 (A)
- net at A1.D49: now also D3.2 (A)
- net BGND: now reaches A1.GND2 (GND)
- net BGND: now also J1.1 (Pin_1)
- net Speaker_GND: now reaches A1.GND3 (GND)
- net Speaker_GND: now also C1.1, LS1.2, Q1.1 (E)
- net Ultrasonic_GND: now reaches A1.GND5 (GND)
- net Ultrasonic_GND: now also J2.4 (Pin_4)
- net GND: now reaches A1.GND6 (GND)
- net GND: now also J3.2, J3.3, J4.3 (Pin_3), J5.6 (Pin_6), J8.2 (Pin_2), R4.2, R5.2, R6.2, R7.1, R8.1, U1.2 (IN+), U1.4 (OUT-)
- removed net +5V: A1.5V1 (5V), A1.5V3 (5V), A1.GND1 (GND), C1.1, LS1.2, Q1.1 (E), R2.2
- new net: D3.1 (K), R6.1
- new net: J7.2 (Pin_2), R8.2
- new net: J6.2 (Pin_2), R7.2
- new net: D1.1 (K), R4.1
- new net +5V Matrix: J8.1 (Pin_1), U1.3 (OUT-)
- new net +5V_Speaker: A1.5V3 (5V), R2.2
- new net +5V_Ultrasonic: A1.5V1 (5V)
- new net +5v_Ultrasonic: J2.1 (Pin_1)
- new net R2: J1.12 (Pin_12)
- new net YGND: A1.GND1 (GND), J1.13 (Pin_13)
Other:
- note added: "12v-5v_Regulator"
- moved on the sheet: A1, C1, C2, LS1, Q1, R1, R2, R3

Commit message: Add files via upload
Parts:
- removed J8: Waveshare_PWR, Connector_PinHeader_1.00mm:PinHeader_1x02_P1.00mm_Vertical, symbol Connector_Generic:Conn_01x02
- removed LS1: Speaker, Buzzer_Beeper:Speaker_CUI_CMR-1206S-67, symbol Device:Speaker
- removed R8: R10k, Resistor_SMD:R_0805_2012Metric_Pad1.20x1.40mm_HandSolder, symbol Device:R
- added J9: WAVESHARE_PWR, Connector_Molex:Molex_KK-396_5273-04A_1x04_P3.96mm_Vertical, symbol Connector_Generic:Conn_01x04
- added LS1: Speaker, Connector_PinHeader_1.00mm:PinHeader_1x02_P1.00mm_Vertical, symbol Connector_Generic:Conn_01x02
- added R9: 10k, Resistor_SMD:R_0805_2012Metric_Pad1.20x1.40mm_HandSolder, symbol Device:R
- D1, D2, D3: footprint LED_THT:LED_D5.0mm_Horizontal_O6.35mm_Z15.0mm -> LED_THT:LED_D5.0mm
- J3: value Barrel_Jack_Switch_Pin3Ring -> PJ-102AH
- J5: footprint (none) -> Connector_PinHeader_1.00mm:PinHeader_1x06_P1.00mm_Vertical
- J6: value Button0 -> Button_Conn
- J7: value Button1 -> Button_Conn
- Q1: footprint Package_TO_SOT_THT:TO-18-3 -> Package_TO_SOT_SMD:SOT-23_Handsoldering
- R1: value R220 -> 220
- R2: value R20 -> 20
- R3: value R100 -> 100
- R4, R5, R6: value R600 -> 600
- R7: value R10k -> 10k
Connections:
- net +5V_Speaker is gone; now on net +5V: A1.5V3 (5V), R2.2
- net +5V_Ultrasonic is gone; now on net +5V: A1.5V1 (5V)
- net +5v_Ultrasonic is gone; now on net +5V: J2.1 (Pin_1)
- net BGND is gone; now on net GND: A1.GND2 (GND), J1.1 (Pin_1)
- net Speaker_GND is gone; now on net GND: A1.GND3 (GND), C1.1, Q1.1 (E)
- net Ultrasonic_GND is gone; now on net GND: A1.GND5 (GND), J2.4 (Pin_4)
- net YGND is gone; now on net GND: A1.GND1 (GND), J1.13 (Pin_13)
- net +12V: now also A1.VIN; no longer J3.1, J4.1 (Pin_1)
- net Button0: now also R9.1
- net Button1: now also R7.1
- net GND: now also A1.GND4 (SPI_GND), J6.2 (Pin_2), J7.2 (Pin_2), J9.3 (Pin_3), J9.4 (Pin_4), LS1.2 (Pin_2); no longer R7.1
- net R1: no longer A1.D27
- net R2: now also A1.D27
- net at C2.2: now also LS1.1 (Pin_1)
- net +5V: now reaches R7.2
- net +5V: now also A1.5V2 (SPI_5V), A1.5V4 (5V), J9.1 (Pin_1), J9.2 (Pin_2), R9.2; no longer J6.2 (Pin_2)
- net +5V Matrix renamed +5V_Matrix
- new net 12V_SWITCH: J3.1, J4.1 (Pin_1)
Other:
- note added: "1738-DFR0831-ND"
- note removed: "12v-5v_Regulator"
- moved on the sheet: J4, J6

Commit message: Add files via upload
Parts:
- J1: value Waveshare_Input_Conn -> WAVESHARE_INPUT_CONN
- J2: value Ultrasonic_Conn -> ULTRASON_CONN
- J4: value LED_Switch_Conn -> LED_SWITCH_CON
- J5: value Debug_Conn -> DEBUG_CONN
- J6, J7: value Button_Conn -> BUTTON_CONN
- LS1: value Speaker -> SPEAKER
Connections:
- net +5V_Matrix renamed +5V_MATRIX
- net Button0 renamed BUTTON_1
- net Button1 renamed BUTTON_2
- net Echo renamed ECHO
- net Speaker_PWM renamed SPEAKER_PWM
- net Trig renamed TRIG
Other:
- moved on the sheet: U1
Changed lines of the file:
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@@
 	)
 	(junction
+		(at 200.66 105.41)
+		(diameter 0)
+		(color 0 0 0 0)
+	)
+	(junction
 		(at 39.37 170.18)
 		(diameter 0)
@@
 	(wire
 		(pts
-			(xy 251.46 120.65) (xy 260.35 120.65)
+			(xy 248.92 120.65) (xy 260.35 120.65)
 		)
 		(stroke
@@
 	(wire
 		(pts
-			(xy 214.63 109.22) (xy 218.44 109.22)
+			(xy 199.39 105.41) (xy 200.66 105.41)
 		)
 		(stroke
@@
 	(wire
 		(pts
-			(xy 173.99 92.71) (xy 173.99 93.98)
+			(xy 180.34 99.06) (xy 180.34 100.33)
 		)
 		(stroke
@@
 	(wire
 		(pts
+			(xy 200.66 105.41) (xy 203.2 105.41)
+		)
+		(stroke
+			(width 0)
+			(type default)
+		)
+	)
+	(wire
+		(pts
 			(xy 129.54 64.77) (xy 132.08 64.77)
 		)
@@
 	(wire
 		(pts
-			(xy 240.03 82.55) (xy 248.92 82.55)
+			(xy 237.49 82.55) (xy 248.92 82.55)
 		)
 		(stroke
@@
 	(wire
 		(pts
-			(xy 173.99 93.98) (xy 179.07 93.98)
+			(xy 180.34 100.33) (xy 185.42 100.33)
 		)
 		(stroke
@@
 	(wire
 		(pts
-			(xy 105.41 93.98) (xy 113.03 93.98)
+			(xy 105.41 93.98) (xy 114.3 93.98)
 		)
 		(stroke
@@
 	(wire
 		(pts
-			(xy 218.44 92.71) (xy 218.44 93.98)
+			(xy 204.47 99.06) (xy 204.47 100.33)
 		)
 		(stroke
@@
 	(wire
 		(pts
-			(xy 175.26 109.22) (xy 179.07 109.22)
+			(xy 181.61 105.41) (xy 185.42 105.41)
 		)
 		(stroke
@@
 	(wire
 		(pts
-			(xy 134.62 99.06) (xy 138.43 99.06)
+			(xy 133.35 99.06) (xy 138.43 99.06)
 		)
 		(stroke
@@
 	(wire
 		(pts
-			(xy 105.41 152.4) (xy 116.84 152.4)
+			(xy 105.41 152.4) (xy 119.38 152.4)
 		)
 		(stroke
@@
 	(wire
 		(pts
-			(xy 105.41 96.52) (xy 113.03 96.52)
+			(xy 105.41 96.52) (xy 114.3 96.52)
 		)
 		(stroke
@@
 	(wire
 		(pts
-			(xy 214.63 93.98) (xy 218.44 93.98)
+			(xy 200.66 100.33) (xy 204.47 100.33)
 		)
 		(stroke
@@
 	(wire
 		(pts
-			(xy 134.62 96.52) (xy 138.43 96.52)
+			(xy 133.35 96.52) (xy 138.43 96.52)
 		)
 		(stroke
@@
 	(text "	\n1738-DFR0831-ND"
 		(exclude_from_sim no)
-		(at 197.104 89.154 0)
+		(at 193.548 94.742 0)
 		(effects
 			(font
@@
 		)
 	)
-	(label "Echo"
-		(at 134.62 99.06 0)
+	(label "ECHO"
+		(at 133.35 99.06 0)
 		(fields_autoplaced yes)
 		(effects
@@
 		)
 	)
-	(label "Speaker_PWM"
-		(at 116.84 152.4 180)
+	(label "SPEAKER_PWM"
+		(at 119.38 152.4 180)
 		(fields_autoplaced yes)
 		(effects
@@
 		)
 	)
-	(label "Trig"
-		(at 134.62 96.52 0)
+	(label "TRIG"
+		(at 133.35 96.52 0)
 		(fields_autoplaced yes)
 		(effects
@@
 		)
 	)
-	(label "Speaker_PWM"
+	(label "SPEAKER_PWM"
 		(at 200.66 149.86 0)
 		(fields_autoplaced yes)
@@
 		)
 	)
-	(label "Echo"
+	(label "ECHO"
 		(at 110.49 124.46 180)
 		(fields_autoplaced yes)
@@
 		)
 	)
-	(label "Button1"
-		(at 251.46 120.65 0)
+	(label "BUTTON_2"
+		(at 248.92 120.65 0)
 		(fields_autoplaced yes)
 		(effects
@@
 		)
 	)
-	(label "Button1"
-		(at 113.03 96.52 180)
+	(label "BUTTON_2"
+		(at 114.3 96.52 180)
 		(fields_autoplaced yes)
 		(effects
@@
 		)
 	)
-	(label "Trig"
+	(label "TRIG"
 		(at 110.49 121.92 180)
 		(fields_autoplaced yes)
@@
 		)
 	)
-	(label "Button0"
-		(at 240.03 82.55 0)
+	(label "BUTTON_1"
+		(at 237.49 82.55 0)
 		(fields_autoplaced yes)
 		(effects
@@
 		)
 	)
-	(label "Button0"
-		(at 113.03 93.98 180)
+	(label "BUTTON_1"
+		(at 114.3 93.98 180)
 		(fields_autoplaced yes)
 		(effects
@@
 	(symbol
 		(lib_id "power:GND")
-		(at 218.44 109.22 0)
+		(at 203.2 105.41 0)
 		(unit 1)
 		(exclude_from_sim no)
@@
 		(fields_autoplaced yes)
 		(property "Reference" "#PWR020"
-			(at 218.44 115.57 0)
+			(at 203.2 111.76 0)
 			(effects
 				(font
@@
 		)
 		(property "Value" "GND"
-			(at 218.44 114.3 0)
+			(at 203.2 110.49 0)
 			(effects
 				(font
@@
 		)
 		(property "Footprint" ""
-			(at 218.44 109.22 0)
+			(at 203.2 105.41 0)
 			(effects
 				(font
@@
 		)
 		(property "Datasheet" ""
-			(at 218.44 109.22 0)
+			(at 203.2 105.41 0)
 			(effects
 				(font
@@
 		)
 		(property "Description" "Power symbol creates a global label with name \"GND\" , ground"
-			(at 218.44 109.22 0)
+			(at 203.2 105.41 0)
 			(effects
 				(font
@@
 	(symbol
 		(lib_id "power:GND")
-		(at 175.26 109.22 0)
+		(at 181.61 105.41 0)
 		(unit 1)
 		(exclude_from_sim no)
@@
 		(fields_autoplaced yes)
 		(property "Reference" "#PWR019"
-			(at 175.26 115.57 0)
+			(at 181.61 111.76 0)
 			(effects
 				(font
@@
 		)
 		(property "Value" "GND"
-			(at 175.26 114.3 0)
+			(at 181.61 110.49 0)
 			(effects
 				(font
@@
 		)
 		(property "Footprint" ""
-			(at 175.26 109.22 0)
+			(at 181.61 105.41 0)
 			(effects
 				(font
@@
 		)
 		(property "Datasheet" ""
-			(at 175.26 109.22 0)
+			(at 181.61 105.41 0)
 			(effects
 				(font
@@
 		)
 		(property "Description" "Power symbol creates a global label with name \"GND\" , ground"
-			(at 175.26 109.22 0)
+			(at 181.61 105.41 0)
 			(effects
 				(font
@@
 			)
 		)
-		(property "Value" "LED_Switch_Conn"
+		(property "Value" "LED_SWITCH_CON"
 			(at 227.33 66.0399 0)
 			(effects
@@
 			)
 		)
-		(property "Value" "Ultrasonic_Conn"
+		(property "Value" "ULTRASON_CONN"
 			(at 146.05 99.0599 0)
 			(effects
@@
 			)
 		)
-		(property "Value" "Debug_Conn"
+		(property "Value" "DEBUG_CONN"
 			(at 119.38 139.6999 0)
 			(effects
@@
 			)
 		)
-		(property "Value" "Waveshare_Input_Conn"
+		(property "Value" "WAVESHARE_INPUT_CONN"
 			(at 138.43 55.88 0)
 			(effects
@@
 			)
 		)
-		(property "Value" "Speaker"
+		(property "Value" "SPEAKER"
 			(at 261.62 147.3199 0)
 			(effects
@@
 			)
 		)
-		(property "Value" "Button_Conn"
+		(property "Value" "BUTTON_CONN"
 			(at 256.54 85.0899 0)
 			(effects
@@
 	(symbol
 		(lib_id "power:+5V")
-		(at 218.44 92.71 0)
+		(at 204.47 99.06 0)
 		(unit 1)
 		(exclude_from_sim no)
@@
 		(dnp no)
 		(property "Reference" "#PWR07"
-			(at 218.44 96.52 0)
+			(at 204.47 102.87 0)
 			(effects
 				(font
@@
 			)
 		)
-		(property "Value" "+5V_Matrix"
-			(at 213.106 88.646 0)
+		(property "Value" "+5V_MATRIX"
+			(at 204.724 99.822 0)
 			(effects
 				(font
@@
 		)
 		(property "Footprint" ""
-			(at 218.44 92.71 0)
+			(at 204.47 99.06 0)
 			(effects
 				(font
@@
 		)
 		(property "Datasheet" ""
-			(at 218.44 92.71 0)
+			(at 204.47 99.06 0)
 			(effects
 				(font
@@
 		)
 		(property "Description" "Power symbol creates a global label with name \"+5V\""
-			(at 218.44 92.71 0)
+			(at 204.47 99.06 0)
 			(effects
 				(font
@@
 			)
 		)
-		(property "Value" "Button_Conn"
+		(property "Value" "BUTTON_CONN"
 			(at 267.97 123.1899 0)
 			(effects
@@
 	(symbol
 		(lib_id "Matrix_Board_Lib:DFR0831")
-		(at 196.85 101.6 0)
+		(at 203.2 107.95 0)
 		(unit 1)
 		(exclude_from_sim no)
@@
 		(dnp no)
 		(property "Reference" "U1"
-			(at 196.85 87.122 0)
+			(at 193.294 92.71 0)
 			(effects
 				(font
@@
 		)
 		(property "Value" "~"
-			(at 188.595 90.17 0)
+			(at 194.945 96.52 0)
 			(effects
 				(font
@@
 		)
 		(property "Footprint" "matrixboard:DFR_Regulator"
-			(at 157.48 114.3 0)
+			(at 163.83 120.65 0)
 			(effects
 				(font
@@
 		)
 		(property "Datasheet" ""
-			(at 157.48 114.3 0)
+			(at 163.83 120.65 0)
 			(effects
 				(font
@@
 		)
 		(property "Description" ""
-			(at 157.48 114.3 0)
+			(at 163.83 120.65 0)
 			(effects
 				(font
@@
 	(symbol
 		(lib_id "power:+12V")
-		(at 173.99 92.71 0)
+		(at 180.34 99.06 0)
 		(unit 1)
 		(exclude_from_sim no)
@@
 		(dnp no)
 		(property "Reference" "#PWR03"
-			(at 173.99 96.52 0)
+			(at 180.34 102.87 0)
 			(effects
 				(font
@@
 		)
 		(property "Value" "+12V"
-			(at 171.45 88.138 0)
+			(at 173.228 99.568 0)
 			(effects
 				(font
@@
 		)
 		(property "Footprint" ""
-			(at 173.99 92.71 0)
+			(at 180.34 99.06 0)
 			(effects
 				(font
@@
 		)
 		(property "Datasheet" ""
-			(at 173.99 92.71 0)
+			(at 180.34 99.06 0)
 			(effects
 				(font
@@
 		)
 		(property "Description" "Power symbol creates a global label with name \"+12V\""
-			(at 173.99 92.71 0)
+			(at 180.34 99.06 0)
 			(effects
 				(font
